Commit message: added camera_link

File: mz07l_description/urdf/mz07L_dual.urdf (robot description, URDF)
Before this commit: robot mz07L, 9 links, 8 joints
Links:
- added link camera_link
Joints:
- added joint camera_joint: type fixed, parent gripper, child camera_link, origin xyz=-0.095 0 0.22 rpy=0 -1.57079632679 0

Commit message: used xacro urdf nachi

File: mz07l_description/urdf/mz07L_dual.urdf (robot description, URDF)
Before this commit: robot mz07L, 10 links, 9 joints
Links:
- added link ultrasonic_link
Joints:
- added joint ultrasonic_joint: type fixed, parent tcp, child ultrasonic_link, origin xyz=0 0 -0.08 rpy=0 -1.57079632679 0
- joint camera_joint: origin xyz=-0.095 0 0.22 rpy=0 -1.57079632679 0 -> xyz=-0.13 0 0.175 rpy=0 -1.57079632679 0
- joint tcp_joint: origin xyz=0 0 0.2702 rpy=0 0 0 -> xyz=0 0 0.265 rpy=0 0 0
